Commit message: fix: align demo with gazebo classic runtime

File: src/robot_lab_description/urdf/lab_ur_mecanum.urdf.xacro (robot description, xacro)
@@ -22,5 +22,4 @@
   <xacro:arg name="ros_namespace" default=""/>
   <xacro:include filename="$(find ur_description)/urdf/ur_macro.xacro"/>
-  <xacro:include filename="$(find ur_description)/urdf/inc/ur_joint_control.xacro"/>
   <xacro:include filename="$(find robot_lab_description)/urdf/inc/parallel_gripper_macro.xacro"/>
   <xacro:include filename="$(find robot_lab_description)/urdf/inc/mecanum_base_macro.xacro"/>
@@ -36,6 +35,5 @@
     safety_limits="$(arg safety_limits)"
     safety_pos_margin="$(arg safety_pos_margin)"
-    safety_k_position="$(arg safety_k_position)"
-    force_abs_paths="true">
+    safety_k_position="$(arg safety_k_position)">
     <origin xyz="0 0 0" rpy="0 0 0"/>
   </xacro:ur_robot>
@@ -45,5 +43,34 @@
       <plugin>gz_ros2_control/GazeboSimSystem</plugin>
     </hardware>
-    <xacro:ur_joint_control_description tf_prefix="$(arg tf_prefix)"/>
+    <joint name="$(arg tf_prefix)shoulder_pan_joint">
+      <command_interface name="position"/>
+      <state_interface name="position"/>
+      <state_interface name="velocity"/>
+    </joint>
+    <joint name="$(arg tf_prefix)shoulder_lift_joint">
+      <command_interface name="position"/>
+      <state_interface name="position"/>
+      <state_interface name="velocity"/>
+    </joint>
+    <joint name="$(arg tf_prefix)elbow_joint">
+      <command_interface name="position"/>
+      <state_interface name="position"/>
+      <state_interface name="velocity"/>
+    </joint>
+    <joint name="$(arg tf_prefix)wrist_1_joint">
+      <command_interface name="position"/>
+      <state_interface name="position"/>
+      <state_interface name="velocity"/>
+    </joint>
+    <joint name="$(arg tf_prefix)wrist_2_joint">
+      <command_interface name="position"/>
+      <state_interface name="position"/>
+      <state_interface name="velocity"/>
+    </joint>
+    <joint name="$(arg tf_prefix)wrist_3_joint">
+      <command_interface name="position"/>
+      <state_interface name="position"/>
+      <state_interface name="velocity"/>
+    </joint>
     <joint name="$(arg tf_prefix)gripper_left_finger_joint">
       <command_interface name="position"/>
